File: AVI_Computer.kicad_sch (KiCad schematic)
At the start: 14 parts, among them IC1 ESP32-S2-MINI-2U-N4, IC2 LM3671MF-3.3_NOPB, IC3 LM3671MF-3.3_NOPB, IC4 BMP390, IC5 BMI270, J1 USB4105-GF-A-060

Commit message: cghanges
Parts:
- added J2: Conn_01x06_Pin, symbol Connector:Conn_01x06_Pin
- added J3: Conn_01x03_Pin, symbol Connector:Conn_01x03_Pin
Connections:
- net +5V: now also J1.A4 (VBUS), J1.A9 (VBUS), J1.B4 (VBUS), J1.B9 (VBUS)
- net GND: now also J2.6 (Pin_6), J3.3 (Pin_3)
- new net +3.3V: J2.1 (Pin_1), J3.1 (Pin_1)
- new net CLK: J2.4 (Pin_4)
- new net CS: J2.5 (Pin_5)
- new net MISO: J2.3 (Pin_3)
- new net MOSI: J2.2 (Pin_2)
- new net PWM: J3.2 (Pin_2)
Changed lines of the file:
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@@
     (effects (font (size 1.27 1.27)) (justify right bottom))
+  )
+  (label "PWM" (at 97.79 105.41 90) (fields_autoplaced)
+    (effects (font (size 1.27 1.27)) (justify left bottom))
   )
   (label "scl" (at 45.72 102.87 0) (fields_autoplaced)
@@
     (effects (font (size 1.27 1.27)) (justify right bottom))
   )
+  (label "MOSI" (at 66.04 105.41 90) (fields_autoplaced)
+    (effects (font (size 1.27 1.27)) (justify left bottom))
+  )
+  (label "MISO" (at 68.58 105.41 90) (fields_autoplaced)
+    (effects (font (size 1.27 1.27)) (justify left bottom))
+  )
   (label "sda" (at 138.43 43.18 180) (fields_autoplaced)
     (effects (font (size 1.27 1.27)) (justify right bottom))
@@
     (effects (font (size 1.27 1.27)) (justify right bottom))
   )
+  (label "CS" (at 73.66 105.41 90) (fields_autoplaced)
+    (effects (font (size 1.27 1.27)) (justify left bottom))
+  )
+  (label "CLK" (at 71.12 105.41 90) (fields_autoplaced)
+    (effects (font (size 1.27 1.27)) (justify left bottom))
+  )
   (symbol (lib_name "GND_1") (lib_id "power:GND") (at 260.35 50.8 90) (unit 1)
     (in_bom yes) (on_board yes) (dnp no) (fields_autoplaced)
@@
         (path "/b77ce694-07dd-499d-9145-732ac70060b8"
           (reference "#PWR0103") (unit 1)
+        )
+      )
+    )
+  )
+  (symbol (lib_id "power:+3.3V") (at 63.5 105.41 90) (unit 1)
+    (in_bom yes) (on_board yes) (dnp no) (fields_autoplaced)
+    (property "Reference" "#PWR04" (at 67.31 105.41 0)
+      (effects (font (size 1.27 1.27)) hide)
+    )
+    (property "Value" "+3.3V" (at 59.69 106.045 90)
+      (effects (font (size 1.27 1.27)) (justify left))
+    )
+    (property "Footprint" "" (at 63.5 105.41 0)
+      (effects (font (size 1.27 1.27)) hide)
+    )
+    (property "Datasheet" "" (at 63.5 105.41 0)
+      (effects (font (size 1.27 1.27)) hide)
+    )
+    (pin "1")
+    (instances
+      (project "AVI_Computer"
+        (path "/b77ce694-07dd-499d-9145-732ac70060b8"
+          (reference "#PWR04") (unit 1)
         )
       )
@@
     )
   )
+  (symbol (lib_id "Connector:Conn_01x06_Pin") (at 68.58 110.49 90) (unit 1)
+    (in_bom yes) (on_board yes) (dnp no) (fields_autoplaced)
+    (property "Reference" "J2" (at 69.85 113.03 90)
+      (effects (font (size 1.27 1.27)))
+    )
+    (property "Value" "Conn_01x06_Pin" (at 69.85 115.57 90)
+      (effects (font (size 1.27 1.27)))
+    )
+    (property "Footprint" "" (at 68.58 110.49 0)
+      (effects (font (size 1.27 1.27)) hide)
+    )
+    (property "Datasheet" "~" (at 68.58 110.49 0)
+      (effects (font (size 1.27 1.27)) hide)
+    )
+    (pin "1")
+    (pin "2")
+    (pin "3")
+    (pin "4")
+    (pin "5")
+    (pin "6")
+    (instances
+      (project "AVI_Computer"
+        (path "/b77ce694-07dd-499d-9145-732ac70060b8"
+          (reference "J2") (unit 1)
+        )
+      )
+    )
+  )
   (symbol (lib_id "SamacSys_Parts:CBC2012T2R2M") (at 69.85 60.96 0) (unit 1)
     (in_bom yes) (on_board yes) (dnp no) (fields_autoplaced)
@@
         (path "/b77ce694-07dd-499d-9145-732ac70060b8"
           (reference "L2") (unit 1)
+        )
+      )
+    )
+  )
+  (symbol (lib_name "GND_3") (lib_id "power:GND") (at 100.33 105.41 90) (unit 1)
+    (in_bom yes) (on_board yes) (dnp no) (fields_autoplaced)
+    (property "Reference" "#PWR06" (at 106.68 105.41 0)
+      (effects (font (size 1.27 1.27)) hide)
+    )
+    (property "Value" "GND" (at 104.14 106.045 90)
+      (effects (font (size 1.27 1.27)) (justify right))
+    )
+    (property "Footprint" "" (at 100.33 105.41 0)
+      (effects (font (size 1.27 1.27)) hide)
+    )
+    (property "Datasheet" "" (at 100.33 105.41 0)
+      (effects (font (size 1.27 1.27)) hide)
+    )
+    (pin "1")
+    (instances
+      (project "AVI_Computer"
+        (path "/b77ce694-07dd-499d-9145-732ac70060b8"
+          (reference "#PWR06") (unit 1)
         )
       )
@@
     )
   )
+  (symbol (lib_name "+5V_1") (lib_id "power:+5V") (at 237.49 116.84 180) (unit 1)
+    (in_bom yes) (on_board yes) (dnp no) (fields_autoplaced)
+    (property "Reference" "#PWR03" (at 237.49 113.03 0)
+      (effects (font (size 1.27 1.27)) hide)
+    )
+    (property "Value" "+5V" (at 237.49 121.92 0)
+      (effects (font (size 1.27 1.27)))
+    )
+    (property "Footprint" "" (at 237.49 116.84 0)
+      (effects (font (size 1.27 1.27)) hide)
+    )
+    (property "Datasheet" "" (at 237.49 116.84 0)
+      (effects (font (size 1.27 1.27)) hide)
+    )
+    (pin "1")
+    (instances
+      (project "AVI_Computer"
+        (path "/b77ce694-07dd-499d-9145-732ac70060b8"
+          (reference "#PWR03") (unit 1)
+        )
+      )
+    )
+  )
   (symbol (lib_id "power:GND") (at 139.7 30.48 270) (unit 1)
     (in_bom yes) (on_board yes) (dnp no) (fields_autoplaced)
@@
     )
   )
+  (symbol (lib_name "GND_3") (lib_id "power:GND") (at 76.2 105.41 90) (unit 1)
+    (in_bom yes) (on_board yes) (dnp no) (fields_autoplaced)
+    (property "Reference" "#PWR05" (at 82.55 105.41 0)
+      (effects (font (size 1.27 1.27)) hide)
+    )
+    (property "Value" "GND" (at 80.01 106.045 90)
+      (effects (font (size 1.27 1.27)) (justify right))
+    )
+    (property "Footprint" "" (at 76.2 105.41 0)
+      (effects (font (size 1.27 1.27)) hide)
+    )
+    (property "Datasheet" "" (at 76.2 105.41 0)
+      (effects (font (size 1.27 1.27)) hide)
+    )
+    (pin "1")
+    (instances
+      (project "AVI_Computer"
+        (path "/b77ce694-07dd-499d-9145-732ac70060b8"
+          (reference "#PWR05") (unit 1)
+        )
+      )
+    )
+  )
   (symbol (lib_id "power:GND") (at 66.04 154.94 90) (unit 1)
     (in_bom yes) (on_board yes) (dnp no) (fields_autoplaced)
@@
     )
   )
+  (symbol (lib_id "Connector:Conn_01x03_Pin") (at 97.79 110.49 90) (unit 1)
+    (in_bom yes) (on_board yes) (dnp no) (fields_autoplaced)
+    (property "Reference" "J3" (at 97.79 113.03 90)
+      (effects (font (size 1.27 1.27)))
+    )
+    (property "Value" "Conn_01x03_Pin" (at 97.79 115.57 90)
+      (effects (font (size 1.27 1.27)))
+    )
+    (property "Footprint" "" (at 97.79 110.49 0)
+      (effects (font (size 1.27 1.27)) hide)
+    )
+    (property "Datasheet" "~" (at 97.79 110.49 0)
+      (effects (font (size 1.27 1.27)) hide)
+    )
+    (pin "1")
+    (pin "2")
+    (pin "3")
+    (instances
+      (project "AVI_Computer"
+        (path "/b77ce694-07dd-499d-9145-732ac70060b8"
+          (reference "J3") (unit 1)
+        )
+      )
+    )
+  )
   (symbol (lib_id "power:+5V") (at 15.24 30.48 0) (unit 1)
     (in_bom yes) (on_board yes) (dnp no) (fields_autoplaced)
@@
         )
       )
+    )
+  )
+  (symbol (lib_id "power:+3.3V") (at 95.25 105.41 90) (unit 1)
+    (in_bom yes) (on_board yes) (dnp no) (fields_autoplaced)
+    (property "Reference" "#PWR07" (at 99.06 105.41 0)
+      (effects (font (size 1.27 1.27)) hide)
+    )
+    (property "Value" "+3.3V" (at 91.44 106.045 90)
+      (effects (font (size 1.27 1.27)) (justify left))
+    )
+    (property "Footprint" "" (at 95.25 105.41 0)
+      (effects (font (size 1.27 1.27)) hide)
+    )
+    (property "Datasheet" "" (at 95.25 105.41 0)
+      (effects (font (size 1.27 1.27)) hide)
+    )
+    (pin "1")
+    (instances
+      (project "AVI_Computer"
+        (path "/b77ce694-07dd-499d-9145-732ac70060b8"
+          (reference "#PWR07") (unit 1)
+        )
+      )

Commit message: changes
Parts:
- removed J3: Conn_01x03_Pin, symbol Connector:Conn_01x03_Pin
- added J3, J4: Conn_01x02_Pin, symbol Connector:Conn_01x02_Pin
- added Q1, Q2: SSM6K407TU,LF, SOTFL65P210X75-6N, symbol SamacSys_Parts:SSM6K407TU,LF
Connections:
- net 3v3 is gone; now on net +3.3V: C3.1, IC1.3 (3V3), IC2.4 (FB), IC3.4 (FB), IC4.1 (VDDIO), IC4.10 (VDD), IC4.6 (CSB), IC5.12 (CSB), IC5.5 (VDDIO), IC5.8 (VDD), L1.2, L2.2, R3.2, R4.2
- net +3.3V: now also Q1.4 (SOURCE), Q2.4 (SOURCE)
- net GND: now also J3.2 (Pin_2), J4.2 (Pin_2)
- new net Motor1+: J3.1 (Pin_1), Q2.1 (DRAIN_1), Q2.2 (DRAIN_2), Q2.5 (DRAIN_3), Q2.6 (DRAIN_4)
- new net Motor2+: J4.1 (Pin_1), Q1.1 (DRAIN_1), Q1.2 (DRAIN_2), Q1.5 (DRAIN_3), Q1.6 (DRAIN_4)
Other:
- moved on the sheet: J2
