File: AVI_Computer.kicad_pcb (KiCad board)
At the start: 2 copper layers, 14 parts, among them IC1 ESP32-S2-MINI-2U-N4, IC2 LM3671MF-3.3_NOPB, IC3 LM3671MF-3.3_NOPB, IC4 BMP390, IC5 BMI270, J1 USB4105-GF-A-060

Commit message: cghanges
Parts:
- moved R4 37.2 mm to (146.0, 105.2), turned to 90 degrees
- moved L2 34.8 mm to (149.0, 113.5), turned to -90 degrees
- moved L1 34.0 mm to (149.0, 117.5), turned to -90 degrees
- moved IC4 32.3 mm to (145.8, 109.5)
- moved IC2 30.4 mm to (145.8, 117.5)
- moved IC5 28.7 mm to (150.0, 109.5)
- moved IC3 27.6 mm to (145.8, 113.5)
- moved C3 25.2 mm to (151.2, 114.0), turned to 90 degrees
- moved R3 25.0 mm to (149.5, 105.2), turned to 90 degrees
- moved C1 25.0 mm to (149.2, 120.5)
- moved R2 10.1 mm to (153.5, 120.5)
- moved J1 9.36 mm to (160.8, 124.2)
- moved R1 5.85 mm to (168.0, 120.5)
Connections:
- IC1 pad 5: unconnected-(IC1-IO1-Pad5) -> /scl
- IC1 pad 6: unconnected-(IC1-IO2-Pad6) -> /sda
Routing:
- net /3v3: track 0.00 -> 45.0 mm, vias 0 -> 2
- net /scl: track 0.00 -> 21.9 mm
- net /sda: track 0.00 -> 21.4 mm
- net +5V: track 0.00 -> 13.3 mm
- net Net-(J1-CC1): track 0.00 -> 6.28 mm
- net Net-(J1-CC2): track 0.00 -> 6.00 mm
- net /D+: track 0.00 -> 3.08 mm
- net /D-: track 0.00 -> 2.99 mm
- net Net-(IC3-SW): track 0.00 -> 1.97 mm
- net Net-(IC2-SW): track 0.00 -> 1.97 mm
- added copper zone on F.Cu, net GND
Other:
- board outline added: 30 x 30 mm

Commit message: do this and that
Parts:
- added J2: Conn_01x06_Pin, Connector_PinHeader_2.54mm:PinHeader_1x06_P2.54mm_Vertical, F.Cu at (171.5, 103.7)
- added J3: Conn_01x02_Pin, Connector_PinHeader_2.54mm:PinHeader_1x02_P2.54mm_Vertical, F.Cu at (145.5, 127.0)
- added J4: Conn_01x02_Pin, Connector_PinHeader_2.54mm:PinHeader_1x02_P2.54mm_Vertical, F.Cu at (150.2, 127.0)
- added J5: Conn_01x02_Pin, Connector_PinHeader_2.54mm:PinHeader_1x02_P2.54mm_Vertical, F.Cu at (168.2, 124.2)
- added Q1: SSM6K407TU,LF, SamacSys_Parts:SOTFL65P210X75-6N, F.Cu at (150.2, 123.8)
- added Q2: SSM6K407TU,LF, SamacSys_Parts:SOTFL65P210X75-6N, F.Cu at (145.5, 123.8)
- moved C1 3.50 mm to (145.8, 120.5)
- moved R4 1.12 mm to (145.6, 104.2)
- moved R3 1.05 mm to (149.5, 104.2)
- moved IC5 0.92 mm to (149.8, 108.6)
- moved IC4 0.86 mm to (145.7, 108.7)
Connections:
- net /3v3 renamed +3.3V
- IC1 pad 14: unconnected-(IC1-IO10-Pad14) -> /CS
- IC1 pad 15: unconnected-(IC1-IO11-Pad15) -> /MOSI
- IC1 pad 16: unconnected-(IC1-IO12-Pad16) -> /CLK
- IC1 pad 17: unconnected-(IC1-IO13-Pad17) -> /MISO
- IC1 pad 7: unconnected-(IC1-IO3-Pad7) -> Net-(IC1-IO3)
- IC1 pad 8: unconnected-(IC1-IO4-Pad8) -> Net-(IC1-IO4)
- J1 pad A4: Net-(J1-VBUS-PadA4) -> +5V
- J1 pad A9: Net-(J1-VBUS-PadA4) -> +5V
- J1 pad B4: Net-(J1-VBUS-PadA4) -> +5V
- J1 pad B9: Net-(J1-VBUS-PadA4) -> +5V
Routing:
- net +3.3V: track 45.0 -> 86.4 mm, vias 2 -> 3
- net /CS: track 0.00 -> 34.2 mm, vias 0 -> 2
- net Net-(IC1-IO3): track 0.00 -> 28.1 mm, vias 0 -> 2
- net +5V: track 13.3 -> 41.1 mm, vias 0 -> 2
- net /MOSI: track 0.00 -> 21.9 mm, vias 0 -> 2
- net Net-(IC1-IO4): track 0.00 -> 21.7 mm, vias 0 -> 2
- net /CLK: track 0.00 -> 20.1 mm, vias 0 -> 2
- net /MISO: track 0.00 -> 19.6 mm, vias 0 -> 2
- net GND: track 0.00 -> 17.0 mm, vias 0 -> 4
- net /scl: track 21.9 -> 13.4 mm
- net /Motor1+: track 0.00 -> 7.90 mm
- net /Motor2+: track 0.00 -> 7.86 mm
- net /sda: track 21.4 -> 14.8 mm, vias 0 -> 4
Other:
- outline, holes or cut-outs redrawn
