File: PCB/AVI_Computer.kicad_sch (KiCad schematic)
At the start: 20 parts, among them IC1 ESP32-S2-MINI-2U-N4, IC2 LM3671MF-3.3_NOPB, IC3 LM3671MF-3.3_NOPB, IC4 BMP390, IC5 BMI270, J1 USB4105-GF-A-060, J2 Conn_01x06_Pin, J3 Conn_01x02_Pin, J4 Conn_01x02_Pin, J5 Conn_01x02_Pin, Q1 SSM6K407TU,LF, Q2 SSM6K407TU,LF

Commit message: updates
Parts:
- removed IC3: LM3671MF-3.3_NOPB, mouser:SOT95P284X119-5N, symbol SamacSys_Parts:LM3671MF-3.3_NOPB
- removed L2: CBC2012T2R2M, mouser:INDC2012X145N, symbol SamacSys_Parts:CBC2012T2R2M
Connections:
- net GND: no longer J1.S1 (SHIELD)
Other:
- moved on the sheet: C3

Commit message: update
Parts:
- removed C1: EMK316B7475KL-T, mouser:CAPC3216X180N, symbol SamacSys_Parts:EMK316B7475KL-T
- removed C3: TMK212BBJ106KG-T, mouser:CAPC2114X145N, symbol SamacSys_Parts:TMK212BBJ106KG-T
- removed IC1: ESP32-S2-MINI-2U-N4, mouser:ESP32S2MINI2UN4, symbol SamacSys_Parts:ESP32-S2-MINI-2U-N4
- removed IC2: LM3671MF-3.3_NOPB, mouser:SOT95P284X119-5N, symbol SamacSys_Parts:LM3671MF-3.3_NOPB
- removed J1: USB4105-GF-A-060, Connector_USB:USB_C_Receptacle_GCT_USB4105-xx-A_16P_TopMnt_Horizontal, symbol Connector:USB_C_Receptacle
- removed J5: Conn_01x02_Pin, Connector_PinHeader_2.54mm:PinHeader_1x02_P2.54mm_Vertical, symbol Connector:Conn_01x02_Pin
- removed L1: CBC2012T2R2M, mouser:INDC2012X145N, symbol SamacSys_Parts:CBC2012T2R2M
- removed R1, R2: CR0805-FX-5101ELF, RESC2012X60N, symbol SamacSys_Parts:CR0805-FX-5101ELF
Connections:
- net GND: no longer J3.2 (Pin_2)
- new net Motor1-: J3.2 (Pin_2)
